Commit message: world added to simulation

File: realsense/realsense2_description/urdf/_d435.gazebo.xacro (robot description, xacro)
@@ -108,5 +108,5 @@
         <always_on>1</always_on>
         <update_rate>90</update_rate>
-        <visualize>0</visualize>
+        <visualize>1</visualize>
       </sensor>
     </gazebo>
@@ -131,5 +131,5 @@
       	<rangeMinDepth>0.2</rangeMinDepth>
       	<rangeMaxDepth>10.0</rangeMaxDepth>
-      	<pointCloud>false</pointCloud>
+      	<pointCloud>true</pointCloud>
       	<pointCloudTopicName>depth/points</pointCloudTopicName>
       	<pointCloudCutoff>0.5</pointCloudCutoff>

File: robot_setup_sim_description/urdf/setup.urdf (robot description, URDF)
Before this commit: robot setup, 13 links, 12 joints
Links:
- added link left_camera_bottom_screw_frame
- added link left_camera_color_frame
- added link left_camera_color_optical_frame
- added link left_camera_depth_frame
- added link left_camera_depth_optical_frame
- added link left_camera_left_ir_frame
- added link left_camera_left_ir_optical_frame
- added link left_camera_link, mass 0.564; collision box size=0.02505 0.09 0.025; visual mesh filename=package://realsense2_description/meshes/d435.dae
- added link left_camera_right_ir_frame
- added link left_camera_right_ir_optical_frame
- added link left_tripod; collision cylinder length=1.4 radius=0.01; visual cylinder length=1.4 radius=0.01
- added link right_camera_bottom_screw_frame
- added link right_camera_color_frame
- added link right_camera_color_optical_frame
- added link right_camera_depth_frame
- added link right_camera_depth_optical_frame
- added link right_camera_left_ir_frame
- added link right_camera_left_ir_optical_frame
- added link right_camera_link, mass 0.564; collision box size=0.02505 0.09 0.025; visual mesh filename=package://realsense2_description/meshes/d435.dae
- added link right_camera_right_ir_frame
- added link right_camera_right_ir_optical_frame
- added link right_tripod; collision cylinder length=1.4 radius=0.01; visual cylinder length=1.4 radius=0.01
- link robot_stand: geometry collision box size=0.50 0.50 1.0; visual box size=0.50 0.50 1.0
Joints:
- added joint left_camera_color_joint: type fixed, parent left_camera_depth_frame, child left_camera_color_frame, origin xyz=0 0.015 0 rpy=0 0 0
- added joint left_camera_color_optical_joint: type fixed, parent left_camera_color_frame, child left_camera_color_optical_frame, origin xyz=0 0 0 rpy=-1.5707963267948966 0 -1.5707963267948966
- added joint left_camera_depth_joint: type fixed, parent left_camera_link, child left_camera_depth_frame, origin xyz=0 0 0 rpy=0 0 0
- added joint left_camera_depth_optical_joint: type fixed, parent left_camera_depth_frame, child left_camera_depth_optical_frame, origin xyz=0 0 0 rpy=-1.5707963267948966 0 -1.5707963267948966
- added joint left_camera_joint: type fixed, parent base_link, child left_camera_bottom_screw_frame, origin xyz=0.0 -0.40 0.40 rpy=0.0 0.5 0.4
- added joint left_camera_left_ir_joint: type fixed, parent left_camera_depth_frame, child left_camera_left_ir_frame, origin xyz=0 0.0 0 rpy=0 0 0
- added joint left_camera_left_ir_optical_joint: type fixed, parent left_camera_left_ir_frame, child left_camera_left_ir_optical_frame, origin xyz=0 0 0 rpy=-1.5707963267948966 0 -1.5707963267948966
- added joint left_camera_link_joint: type fixed, parent left_camera_bottom_screw_frame, child left_camera_link, origin xyz=0 0.0175 0.0125 rpy=0 0 0
- added joint left_camera_right_ir_joint: type fixed, parent left_camera_depth_frame, child left_camera_right_ir_frame, origin xyz=0 -0.05 0 rpy=0 0 0
- added joint left_camera_right_ir_optical_joint: type fixed, parent left_camera_right_ir_frame, child left_camera_right_ir_optical_frame, origin xyz=0 0 0 rpy=-1.5707963267948966 0 -1.5707963267948966
- added joint right_camera_color_joint: type fixed, parent right_camera_depth_frame, child right_camera_color_frame, origin xyz=0 0.015 0 rpy=0 0 0
- added joint right_camera_color_optical_joint: type fixed, parent right_camera_color_frame, child right_camera_color_optical_frame, origin xyz=0 0 0 rpy=-1.5707963267948966 0 -1.5707963267948966
- added joint right_camera_depth_joint: type fixed, parent right_camera_link, child right_camera_depth_frame, origin xyz=0 0 0 rpy=0 0 0
- added joint right_camera_depth_optical_joint: type fixed, parent right_camera_depth_frame, child right_camera_depth_optical_frame, origin xyz=0 0 0 rpy=-1.5707963267948966 0 -1.5707963267948966
- added joint right_camera_joint: type fixed, parent base_link, child right_camera_bottom_screw_frame, origin xyz=0.0 0.40 0.40 rpy=0.0 0.5 -0.4
- added joint right_camera_left_ir_joint: type fixed, parent right_camera_depth_frame, child right_camera_left_ir_frame, origin xyz=0 0.0 0 rpy=0 0 0
- added joint right_camera_left_ir_optical_joint: type fixed, parent right_camera_left_ir_frame, child right_camera_left_ir_optical_frame, origin xyz=0 0 0 rpy=-1.5707963267948966 0 -1.5707963267948966
- added joint right_camera_link_joint: type fixed, parent right_camera_bottom_screw_frame, child right_camera_link, origin xyz=0 0.0175 0.0125 rpy=0 0 0
- added joint right_camera_right_ir_joint: type fixed, parent right_camera_depth_frame, child right_camera_right_ir_frame, origin xyz=0 -0.05 0 rpy=0 0 0
- added joint right_camera_right_ir_optical_joint: type fixed, parent right_camera_right_ir_frame, child right_camera_right_ir_optical_frame, origin xyz=0 0 0 rpy=-1.5707963267948966 0 -1.5707963267948966
- added joint world_left_tripod: type fixed, parent world, child left_tripod, origin xyz=0.0 -0.40 0.7 rpy=0.0 0.0 0.0
- added joint world_right_tripod: type fixed, parent world, child right_tripod, origin xyz=0.0 0.40 0.7 rpy=0.0 0.0 0.0
- joint robot_stand_robot: origin xyz=0.0 0.0 0.25 rpy=0.0 0.0 0.0 -> xyz=0.0 0.0 0.5 rpy=0 0 0
- joint world_robot_stand: origin xyz=0.0 0.0 0.25 rpy=0.0 0.0 0.0 -> xyz=0.0 0.0 0.5 rpy=0 0 0

File: robot_setup_sim_description/urdf/setup.xacro (robot description, xacro)
@@ -16,8 +16,8 @@
   <!-- Stand and World -->
   <link name="robot_stand">
-    <visual><geometry><box size="0.50 0.50 0.50"/></geometry>
+    <visual><geometry><box size="0.50 0.50 1.0"/></geometry>
       <material name="black_metal"><color rgba="0.1 0.1 0.1 1"/></material>
     </visual>
-    <collision><geometry><box size="0.50 0.50 0.50"/></geometry></collision>
+    <collision><geometry><box size="0.50 0.50 1.0"/></geometry></collision>
   </link>
   <link name="world"/>
@@ -25,17 +25,67 @@
     <parent link="world"/>
     <child link="robot_stand"/>
-    <origin xyz="0.0 0.0 0.25" rpy="0 0 0"/>
+    <origin xyz="0.0 0.0 0.5" rpy="0 0 0"/>
   </joint>
   <joint name="robot_stand_robot" type="fixed">
     <parent link="robot_stand"/>
     <child link="base_link"/>
-    <origin xyz="0.0 0.0 0.25" rpy="0 0 0"/>
+    <origin xyz="0.0 0.0 0.5" rpy="0 0 0"/>
   </joint>
   <xacro:include filename="$(find realsense2_description)/urdf/_d435.urdf.xacro"/>
   <xacro:sensor_d435 name="left_camera" topics_ns="left_camera" parent="base_link">
-    <origin xyz="0.0 -0.40 0.40" rpy="0.0 0.0 0.0"/>
+    <origin xyz="0.0 -0.40 0.40" rpy="0.0 0.5 0.4"/>
   </xacro:sensor_d435>
   <xacro:sensor_d435 name="right_camera" topics_ns="right_camera" parent="base_link">
-    <origin xyz="0.0 0.40 0.40" rpy="0.0 0.0 0.0"/>
+    <origin xyz="0.0 0.40 0.40" rpy="0.0 0.5 -0.4"/>
   </xacro:sensor_d435>
+  <link name="left_tripod">
+  <visual>
+    <geometry>
+      <cylinder radius="0.02" length="1.4"/>
+      <material name="black_metal">
+        <color rgba="0.1 0.1 0.1 1"/>
+      </material>
+    </geometry>
+  </visual>
+  <collision>
+    <geometry>
+      <cylinder radius="0.02" length="1.4"/>
+    </geometry>
+  </collision>
+  <inertial>
+    <origin xyz="0.0 0.0 0.0" rpy="0.0 0.0 0.0"/>
+    <mass value="0.5"/>
+    <inertia ixx="0.0" ixy="0.0" ixz="0.0" iyy="0.0" iyz="0.0" izz="0.0"/>
+  </inertial>
+  </link>
+  <link name="right_tripod">
+  <visual>
+    <geometry>
+      <cylinder radius="0.02" length="1.4"/>
+      <material name="black_metal">
+        <color rgba="0.1 0.1 0.1 1"/>
+      </material>
+    </geometry>
+  </visual>
+  <collision>
+    <geometry>
+      <cylinder radius="0.02" length="1.4"/>
+    </geometry>
+  </collision>
+  <inertial>
+    <origin xyz="0.0 0.0 0.0" rpy="0.0 0.0 0.0"/>
+    <mass value="0.5"/>
+    <inertia ixx="0.0" ixy="0.0" ixz="0.0" iyy="0.0" iyz="0.0" izz="0.0"/>
+  </inertial>
+  </link>
+  <joint name="world_left_tripod" type="fixed">
+    <parent link="world"/>
+    <child link="left_tripod"/>
+    <origin xyz="0.0 -0.40 0.7" rpy="0.0 0.0 0.0"/>
+  </joint>
+  <joint name="world_right_tripod" type="fixed">
+    <parent link="world"/>
+    <child link="right_tripod"/>
+    <origin xyz="0.0 0.40 0.7" rpy="0.0 0.0 0.0"/>
+  </joint>
 </robot>
