Commit message: made the tool0 tcp calibratable ig idk, generated a whole new moveit package for the ur16e, need to test that as well, first need to test if the current moveit config accounts for tool0, if it does, then we dont really need the other moveit_config, but nice to know if that works well, so gotta test that too

File: universal_robot/ur_description/urdf/inc/ur16e_macro.xacro (robot description, xacro)
@@ -26,5 +26,8 @@
    safety_limits:=false
    safety_pos_margin:=0.15
-   safety_k_position:=20"
+   safety_k_position:=20
+   tool0_tcp_x:=0.0
+   tool0_tcp_y:=0.0
+   tool0_tcp_z:=0.0"
   >
     <xacro:include filename="$(find ur_description)/urdf/inc/ur_macro.xacro"/>
@@ -39,4 +42,7 @@
       safety_pos_margin="${safety_pos_margin}"
       safety_k_position="${safety_k_position}"
+      tool0_tcp_x="${tool0_tcp_x}"
+      tool0_tcp_y="${tool0_tcp_y}"
+      tool0_tcp_z="${tool0_tcp_z}"
     />
   </xacro:macro>

File: universal_robot/ur_description/urdf/inc/ur_macro.xacro (robot description, xacro)
@@ -53,5 +53,8 @@
     safety_limits:=false
     safety_pos_margin:=0.15
-    safety_k_position:=20"
+    safety_k_position:=20
+    tool0_tcp_x:=0.0
+    tool0_tcp_y=0.0
+    tool0_tcp_z=0.0"
   >
     <!-- Load configuration data from the provided .yaml files -->
@@ -312,5 +315,5 @@
     <joint name="${prefix}flange-tool0" type="fixed">
       <!-- default toolframe: X+ left, Y+ up, Z+ front -->
-      <origin xyz="0 0 0" rpy="${pi/2.0} 0 ${pi/2.0}"/>
+      <origin xyz="${tool0_tcp_x} ${tool0_tcp_y} ${tool0_tcp_z}" rpy="${pi/2.0} 0 ${pi/2.0}"/>
       <parent link="${prefix}flange"/>
       <child link="${prefix}tool0"/>

File: universal_robot/ur_description/urdf/ur.xacro (robot description, xacro)
@@ -17,4 +17,7 @@
    <xacro:arg name="safety_pos_margin" default="0.15"/>
    <xacro:arg name="safety_k_position" default="20"/>
+   <xacro:arg name="tool0_tcp_x" default="0.0"/>
+   <xacro:arg name="tool0_tcp_y" default="0.0"/>
+   <xacro:arg name="tool0_tcp_z" default="0.0"/>
    <!-- arm -->
    <xacro:ur_robot
@@ -27,4 +30,7 @@
      safety_limits="$(arg safety_limits)"
      safety_pos_margin="$(arg safety_pos_margin)"
-     safety_k_position="$(arg safety_k_position)"/>
+     safety_k_position="$(arg safety_k_position)"
+     tool0_tcp_x="$(arg tool0_tcp_x)"
+     tool0_tcp_y="$(arg tool0_tcp_y)"
+     tool0_tcp_z="$(arg tool0_tcp_z)"/>
 </robot>
