Commit message: added fgp velocity computation with sliding window and linear iir filtering

File: robot_setup_sim_description/urdf/setup.urdf (robot description, URDF)
Before this commit: robot setup, 35 links, 34 joints
Links:
- link left_tripod: mass None -> 0.5; geometry collision cylinder length=1.4 radius=0.02; visual cylinder length=1.4 radius=0.02
- link right_tripod: mass None -> 0.5; geometry collision cylinder length=1.4 radius=0.02; visual cylinder length=1.4 radius=0.02
Joints:
- joint flange-tool0: origin xyz=0 0 0 rpy=1.5707963267948966 0 1.5707963267948966 -> xyz=0.0 0.0 0.0  rpy=1.5707963267948966 0 1.5707963267948966
